File: eagle/SL530.brd (EAGLE design)
At the start: 100 x 100 mm, 42 parts, among them IC4 74LVC1G17DBV, IC5 74LVC1G17DBV, U1 LM1117, X1 MC68000

Commit message: Add files via upload
Collected updates combined
Parts:
- OSC1: value X20MHZ -> X24MHZ
Routing:
- net FC1: track 44.8 -> 44.3 mm
- net CLKCPU: track 130.3 -> 130.1 mm, vias 1 -> 5
Other:
- board text added: "Revision 3"
- board text added: "TF530 "Accelerator" - Tachyon Rev https://github.com/TheRealTachyon/tf530"
- board text removed: "Revision 2"
- board text removed: "TerribleFire 530 "Accelerator" (C) 2016 S.J Leary"
