File: eagle/SL530.sch (EAGLE design)
At the start: 42 parts, among them IC4 74LVC1G17DBV, IC5 74LVC1G17DBV, U1 LM1117, X1 MC68000

Commit message: Add files via upload
Collected updates combined
Parts:
- OSC1: value X20MHZ -> X24MHZ
Changed lines of the file:
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@@
 <?xml version="1.0" encoding="utf-8"?>
 <!DOCTYPE eagle SYSTEM "eagle.dtd">
-<eagle version="7.7.0">
+<eagle version="8.1.1">
 <drawing>
 <settings>
@@
 <parts>
 <part name="X1" library="terriblefire" deviceset="MC68000P" device="" value="MC68000"/>
-<part name="OSC1" library="microbuilder" deviceset="OSCILLATOR" device="" value="X20MHZ"/>
+<part name="OSC1" library="microbuilder" deviceset="OSCILLATOR" device="" value="X24MHZ"/>
 <part name="JP1" library="SparkFun-Retired" deviceset="JUMPER-3" device="PTH" value="CLOCKSEL"/>
 <part name="JTAG" library="microbuilder" deviceset="HEADER-1X6" device="ROUND" value="JTAG"/>
